File: gate.kicad_pcb (KiCad board)
At the start: 2 copper layers, 94.9 x 94.7 mm, 4 parts

Commit message: started Schematic
Parts:
- removed the G*** at (144.5, 104.1) (x4)
- added G*** (x4): LOGO, LOGO, F.Cu at (144.5, 104.1)
Changed lines of the file:
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@@
   )
   (page A4)
+  (title_block
+    (title "Doorway to Heaven Badge")
+    (company "Sarif Industries")
+  )
   (layers
     (0 F.Cu signal)
